File: miniplatform.brd (EAGLE design)
At the start: 100 x 80 mm, 7 parts

Commit message: Layout work.
Parts:
- removed SV1: (no value), con-lstb:MA07-1
- added ACCELEROMETER: (no value), con-lstb:MA05-1
- added MOTOR: (no value), con-lstb:MA07-1
- added X1: (no value), con-wago-500:W237-102
- C12, C7: device rcl:C025-025X050 -> rcl:C0805K
- R1: device rcl:0207/10 -> rcl:R0805
- moved U$2 59.8 mm to (16.5, 25.4), flipped to the bottom, turned to 180 degrees
- moved U$1 31.4 mm to (21.6, 44.5)
- moved R1 28.7 mm to (26.7, 14.0), flipped to the bottom
- moved C7 19.7 mm to (26.7, 7.62), flipped to the bottom, turned to 90 degrees
- moved 3.3V_REG 13.0 mm to (17.8, 11.4), flipped to the bottom, turned to 270 degrees
- moved C12 10.9 mm to (26.7, 11.4), flipped to the bottom, turned to 180 degrees
Connections:
- net LEDSTRIP3 renamed IO1
- net LEDSTRIP4 renamed IO2
- net LIGHTLEVEL renamed ANALOG_6
- net RADIO_MISO renamed MISO
- net SOUND_ANALOG renamed ANALOG_1
- net SPOTLIGHT1 renamed PWM1
- net SPOTLIGHT2 renamed PWM2
- net SPOTLIGHT3 renamed PWM3
- net SPOTLIGHT4 renamed PWM4
- net SPOTLIGHT5 renamed PWM5
- net SPOTLIGHT6 renamed ANALOG_2
- removed net EXTRA_IO1: U$1.A4
- removed net EXTRA_IO2: U$1.A5
- removed net LEDSTRIP1: U$1.5
- removed net LEDSTRIP2: U$1.7
- removed net MOTOR_+: SV1.7
- removed net PROXIMITY: U$1.A6
- removed net RADIO_CLOCK: U$2.P$5
- removed net RADIO_MOSI: U$1.14, U$2.P$6
- removed net RADIO_SCK: U$1.16
- removed net VCC_3.3V: U$2.P$2
- new net ACCEL_X: ACCELEROMETER.4, U$1.A4
- new net ACCEL_Y: ACCELEROMETER.3, U$1.A5
- new net ACCEL_Z: ACCELEROMETER.2, U$1.A6
- new net MOTOR_SELECT: MOTOR.4, U$1.5
- new net RESET: U$1.3
- new net TXI: U$1.2
- new net TXO: U$1.1
- new net VCC: MOTOR.7, X1.1
- net +3V3: now also U$2.P$2
- net +5V: now also ACCELEROMETER.5; no longer SV1.4
- net CLOCK: now also MOTOR.3, U$1.16, U$2.P$5; no longer SV1.3
- net GND: now also ACCELEROMETER.1, MOTOR.5, MOTOR.6, X1.2; no longer SV1.5, SV1.6
- net LATCH: now also MOTOR.2, U$1.7; no longer SV1.2
- net MOSI: now also MOTOR.1, U$1.14, U$2.P$6; no longer SV1.1
Other:
- board size 100 x 80 mm -> 40 x 80 mm

Commit message: Tuned layout.
Parts:
- removed R1: 1k, rcl:R0805
- removed X1: (no value), con-wago-500:W237-102
- added JP1, JP2: (no value), SparkFun:1X08
- added JP11, JP12, JP13, JP14, JP15, JP4, JP5, JP6, JP7, JP8, JP9: M01PTH, SparkFun:1X01
- added JP16: (no value), SparkFun:1X05
- added JP3: (no value), SparkFun:1X02_LOCK_LONGPADS
- moved U$2 23.5 mm to (17.8, 1.91), turned to 0 degrees
- moved U$1 22.2 mm to (12.7, 24.1)
- moved MOTOR 21.0 mm to (12.7, 44.5)
- moved C7 17.8 mm to (8.89, 8.26), turned to 0 degrees
- moved ACCELEROMETER 17.6 mm to (12.7, 33.0), turned to 180 degrees
- moved C12 14.3 mm to (12.7, 8.26)
- moved 3.3V_REG 6.96 mm to (11.4, 14.3), turned to 0 degrees
Connections:
- removed net ANALOG_6: U$1.A7
- removed net IO1: U$1.10
- removed net LATCH: MOTOR.2, U$1.7
- removed net MOTOR_SELECT: MOTOR.4, U$1.5
- new net ANALOG_3: U$1.A6
- new net MOTOR_CLOCK: JP1.3, MOTOR.3, U$1.10
- new net MOTOR_DATA: JP1.8, MOTOR.1, U$1.5
- new net MOTOR_LATCH: JP1.6, MOTOR.2, U$1.7
- net +3V3: now also JP6.1, JP9.1; no longer R1.2
- net +5V: now also JP16.5, JP5.1, MOTOR.4
- net ACCEL_Z: now also U$1.A7; no longer U$1.A6
- net ANALOG_1: now also JP2.2
- net ANALOG_2: now also JP2.1
- net CLOCK: now also JP2.5; no longer MOTOR.3
- net GND: now also JP12.1, JP13.1, JP14.1, JP15.1, JP16.1, JP3.1, JP7.1, JP8.1; no longer R1.1, X1.2
- net IO2: now also JP1.2
- net MISO: now also JP2.6
- net MOSI: now also JP2.7; no longer MOTOR.1
- net PWM1: now also JP1.7
- net PWM2: now also JP1.5
- net PWM3: now also JP1.4
- net PWM4: now also JP1.1
- net PWM5: now also JP2.8
- net RADIO_CE: now also JP2.3
- net RADIO_CSN: now also JP2.4
- net RESET: now also JP16.2
- net TXI: now also JP16.3
- net TXO: now also JP16.4
- net VCC: now also JP11.1, JP3.2, JP4.1; no longer X1.1
Routing:
- net GND: track 0.00 -> 2.54 mm
Other:
- board size 40 x 80 mm -> 25 x 50 mm
