File: miniplatform.sch (EAGLE design)
At the start: 7 parts

Commit message: Layout work.
Parts:
- added ACCELEROMETER: (no value), con-lstb:MA05-1
- added X1: (no value), con-wago-500:W237-102
- C12, C7: device rcl:C-EU025-025X050 -> rcl:C-EUC0805K
- R1: device rcl:R-EU_0207/10 -> rcl:R-EU_R0805
- renumbered SV1 to MOTOR
Connections:
- net LEDSTRIP3 renamed IO1
- net LEDSTRIP4 renamed IO2
- net LIGHTLEVEL renamed ANALOG_6
- net RADIO_MISO renamed MISO
- net SOUND_ANALOG renamed ANALOG_1
- net SPOTLIGHT1 renamed PWM1
- net SPOTLIGHT2 renamed PWM2
- net SPOTLIGHT3 renamed PWM3
- net SPOTLIGHT4 renamed PWM4
- net SPOTLIGHT5 renamed PWM5
- net SPOTLIGHT6 renamed ANALOG_2
- removed net EXTRA_IO1: U$1.A4
- removed net EXTRA_IO2: U$1.A5
- removed net LEDSTRIP1: U$1.2
- removed net LEDSTRIP2: U$1.4
- removed net MOTOR_+: MOTOR.7
- removed net PROXIMITY: U$1.A6
- removed net RADIO_CLOCK: U$2.SCK_SERIAL_CLOCK
- removed net RADIO_MOSI: U$1.*11, U$2.MOSI_MASTER_OUT_SLAVE_IN
- removed net RADIO_SCK: U$1.13
- removed net VCC_3.3V: U$2.VCC_3.3V
- new net ACCEL_X: ACCELEROMETER.4, U$1.A4
- new net ACCEL_Y: ACCELEROMETER.3, U$1.A5
- new net ACCEL_Z: ACCELEROMETER.2, U$1.A6
- new net MOTOR_SELECT: MOTOR.4, U$1.2
- new net RESET: U$1.RST
- new net TXI: U$1.RXI
- new net TXO: U$1.TXO
- new net VCC: MOTOR.7, X1-1.KL
- net +3V3: now also U$2.VCC_3.3V
- net +5V: now also ACCELEROMETER.5; no longer MOTOR.4
- net CLOCK: now also U$1.13, U$2.SCK_SERIAL_CLOCK
- net GND: now also ACCELEROMETER.1, X1-2.KL
- net LATCH: now also U$1.4
- net MOSI: now also U$1.*11, U$2.MOSI_MASTER_OUT_SLAVE_IN

Commit message: Tuned layout.
Parts:
- removed R1: 1k, rcl:R-EU_R0805
- removed X1: (no value), con-wago-500:W237-102
- added JP1, JP2: (no value), SparkFun:M081X08
- added JP11, JP12, JP13, JP14, JP15, JP4, JP5, JP6, JP7, JP8, JP9: M01PTH, SparkFun:M01PTH
- added JP16: (no value), SparkFun:M05PTH
- added JP3: (no value), SparkFun:M02LOCK_LONGPADS
Connections:
- removed net ANALOG_6: U$1.A7
- removed net IO1: U$1.7
- removed net LATCH: MOTOR.2, U$1.4
- removed net MOTOR_SELECT: MOTOR.4, U$1.2
- new net ANALOG_3: U$1.A6
- new net MOTOR_CLOCK: JP1.3, MOTOR.3, U$1.7
- new net MOTOR_DATA: JP1.8, MOTOR.1, U$1.2
- new net MOTOR_LATCH: JP1.6, MOTOR.2, U$1.4
- net +3V3: now also JP6.1, JP9.1; no longer R1.2
- net +5V: now also JP16.5, JP5.1, MOTOR.4
- net ACCEL_Z: now also U$1.A7; no longer U$1.A6
- net ANALOG_1: now also JP2.2
- net ANALOG_2: now also JP2.1
- net CLOCK: now also JP2.5; no longer MOTOR.3
- net GND: now also JP12.1, JP13.1, JP14.1, JP15.1, JP16.1, JP3.1, JP7.1, JP8.1; no longer R1.1, X1-2.KL
- net IO2: now also JP1.2
- net MISO: now also JP2.6
- net MOSI: now also JP2.7; no longer MOTOR.1
- net PWM1: now also JP1.7
- net PWM2: now also JP1.5
- net PWM3: now also JP1.4
- net PWM4: now also JP1.1
- net PWM5: now also JP2.8
- net RADIO_CE: now also JP2.3
- net RADIO_CSN: now also JP2.4
- net RESET: now also JP16.2
- net TXI: now also JP16.3
- net TXO: now also JP16.4
- net VCC: now also JP11.1, JP3.2, JP4.1; no longer X1-1.KL
Other:
- note removed: "NOTE: The regulator needs at least a 10mA load to work, and the radio may draw less than that, so we add some extra pulldown on the 3.3V rail."
